Commit message: 3 rovers with simple colors

File: src/mast_ros/worlds/mast_room.world.xacro (robot description, xacro)
@@ -10,4 +10,8 @@
   <xacro:property name="wall_height" value="2"/>
   <xacro:property name="wall_thickness" value="0.1"/>
+  <xacro:property name="floor_color" value="0.6 0.4 0.2 0.0"/>
+  <xacro:property name="wall_color" value="0.0 0.0 0.1 0.0"/>
+  <xacro:property name="cylinder_color" value="0.5 0.0 0.0 0.0"/>
+  <xacro:property name="box_color" value="0.0 0.5 0.0 0.0"/>
     <scene>
       <ambient>0.5 0.5 0.5 1</ambient>
@@ -71,9 +75,6 @@
           </geometry>
           <material>
-            <script>
-              <uri>model://media/materials/scripts</uri>
-              <uri>model://media/materials/textures</uri>
-              <name>CarparkGroundPlane/Image</name>
-            </script>
+						<ambient>${floor_color}</ambient>
+						<diffuse>${floor_color}</diffuse>
           </material>
         </visual>
@@ -100,9 +101,29 @@
           </geometry>
           <material>
-            <script>
-              <uri>model://media/materials/scripts</uri>
-              <uri>model://media/materials/textures</uri>
-              <name>CarparkGroundPlane/Image</name>
-            </script>
+						<ambient>${wall_color}</ambient>
+          </material>
+        </visual>
+      </link>
+    </model>
+    <model name="wall1">
+      <static>true</static>
+      <link name="wall1_link">
+				<pose>${room_width/2} 0 ${wall_height/2} 0 0 0</pose>
+        <collision name="collision">
+          <geometry>
+            <box>
+              <size>${wall_thickness} ${room_length} ${wall_height}</size>
+            </box>
+          </geometry>
+        </collision>
+        <visual name="visual">
+          <cast_shadows>true</cast_shadows>
+          <geometry>
+            <box>
+              <size>${wall_thickness} ${room_length} ${wall_height}</size>
+            </box>
+          </geometry>
+          <material>
+						<ambient>${wall_color}</ambient>
           </material>
         </visual>
@@ -128,9 +149,5 @@
           </geometry>
           <material>
-            <script>
-              <uri>model://media/materials/scripts</uri>
-              <uri>model://media/materials/textures</uri>
-              <name>CarparkGroundPlane/Image</name>
-            </script>
+						<ambient>${wall_color}</ambient>
           </material>
         </visual>
@@ -156,9 +173,5 @@
           </geometry>
           <material>
-            <script>
-              <uri>model://media/materials/scripts</uri>
-              <uri>model://media/materials/textures</uri>
-              <name>CarparkGroundPlane/Image</name>
-            </script>
+						<ambient>${wall_color}</ambient>
           </material>
         </visual>
@@ -184,9 +197,5 @@
           </geometry>
           <material>
-            <script>
-              <uri>model://media/materials/scripts</uri>
-              <uri>model://media/materials/textures</uri>
-              <name>CarparkGroundPlane/Image</name>
-            </script>
+						<ambient>${wall_color}</ambient>
           </material>
         </visual>
@@ -215,9 +224,5 @@
           </geometry>
           <material>
-            <script>
-              <uri>model://media/materials/scripts</uri>
-              <uri>model://media/materials/textures</uri>
-              <name>CarparkGroundPlane/Image</name>
-            </script>
+						<ambient>${cylinder_color}</ambient>
           </material>
         </visual>
@@ -249,9 +254,5 @@
           </geometry>
           <material>
-            <script>
-              <uri>model://media/materials/scripts</uri>
-              <uri>model://media/materials/textures</uri>
-              <name>CarparkGroundPlane/Image</name>
-            </script>
+						<ambient>${box_color}</ambient>
           </material>
         </visual>
@@ -261,5 +262,5 @@
 <xacro:draw_box name="box1"  x="${-room_width/8}" y="${-room_length/8}"
 	length="0.5" width="0.5" height="1"/>
-<xacro:draw_box name="box2"  x="${room_width/8}" y="${-room_length/8}"
+<xacro:draw_box name="box2"  x="${room_width/8}" y="${room_length/8}"
 	length="0.5" width="0.5" height="1"/>
   </world>
